File: electrical/kicad_project/mcu_esp32.kicad_sch (KiCad schematic)
At the start: 4 parts, among them U1 ESP32-WROOM-32

Commit message: commit
Parts:
- added C3: 22µF, symbol Device:C
- added J1: Conn_01x04, symbol Connector_Generic:Conn_01x04
- added R2: 10kΩ, symbol Device:R
- added SW1, SW2: SW_Push, symbol Switch:SW_Push
Connections:
- net +3V3: now also C3.1, J1.3 (Pin_3), R2.1
- net DSHOT_M1: now also U1.16 (IO13); no longer U1.14 (IO12)
- net DSHOT_M2: now also U1.13 (IO14); no longer U1.16 (IO13)
- net DSHOT_M3: now also U1.12 (IO27); no longer U1.13 (IO14)
- net DSHOT_M4: now also U1.8 (IO32); no longer U1.23 (IO15)
- net GND: now also C3.2, J1.4 (Pin_4), SW1.2, SW2.1
- net at C1.1, R1.2, U1.3 (EN): now also SW2.2
- net at U1.25 (IO0): now also R2.2, SW1.1
- net at U1.6 (IO34): now also J1.1 (Pin_1)
- net at U1.7 (IO35): now also J1.2 (Pin_2)
- no-connect marks 24 -> 21
Other:
- moved on the sheet: C1, R1

Commit message: commit
Connections:
- net at U1.34 (RXD0/IO3): now also J1.2 (Pin_2)
- net at U1.35 (TXD0/IO1): now also J1.1 (Pin_1)
- net at U1.6 (IO34): no longer J1.1 (Pin_1)
- net at U1.7 (IO35): no longer J1.2 (Pin_2)
Other:
- moved on the sheet: J1
Changed lines of the file:
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@@
+	)
+	(no_connect
+		(at 110.49 115.57)
 	)
 	(no_connect
@@
 	)
 	(no_connect
-		(at 110.49 62.23)
-	)
-	(no_connect
 		(at 110.49 102.87)
-	)
-	(no_connect
-		(at 110.49 67.31)
 	)
 	(no_connect
@@
 	)
 	(no_connect
+		(at 110.49 118.11)
+	)
+	(no_connect
 		(at 80.01 90.17)
 	)
@@
 	(wire
 		(pts
-			(xy 110.49 118.11) (xy 127 118.11)
-		)
-		(stroke
-			(width 0)
-			(type default)
-		)
-	)
-	(wire
-		(pts
 			(xy 95.25 39.37) (xy 95.25 54.61)
 		)
@@
 	(wire
 		(pts
+			(xy 110.49 67.31) (xy 137.16 67.31)
+		)
+		(stroke
+			(width 0)
+			(type default)
+		)
+	)
+	(wire
+		(pts
 			(xy 101.6 26.67) (xy 101.6 39.37)
 		)
@@
 	(wire
 		(pts
+			(xy 137.16 64.77) (xy 148.59 64.77)
+		)
+		(stroke
+			(width 0)
+			(type default)
+		)
+	)
+	(wire
+		(pts
 			(xy 80.01 59.69) (xy 49.53 59.69)
 		)
@@
 	(wire
 		(pts
-			(xy 110.49 115.57) (xy 127 115.57)
-		)
-		(stroke
-			(width 0)
-			(type default)
-		)
-	)
-	(wire
-		(pts
 			(xy 39.37 68.58) (xy 41.91 68.58)
 		)
@@
 		(pts
 			(xy 81.28 26.67) (xy 74.93 26.67)
+		)
+		(stroke
+			(width 0)
+			(type default)
+		)
+	)
+	(wire
+		(pts
+			(xy 110.49 62.23) (xy 148.59 62.23)
+		)
+		(stroke
+			(width 0)
+			(type default)
+		)
+	)
+	(wire
+		(pts
+			(xy 137.16 67.31) (xy 137.16 64.77)
 		)
 		(stroke
@@
 	(symbol
 		(lib_id "power:+3V3")
-		(at 127 120.65 90)
+		(at 148.59 67.31 90)
 		(unit 1)
 		(body_style 1)
@@
 		(fields_autoplaced yes)
 		(property "Reference" "#PWR07"
-			(at 130.81 120.65 0)
+			(at 152.4 67.31 0)
 			(hide yes)
 			(show_name no)
@@
 		)
 		(property "Value" "+3V3"
-			(at 123.19 120.6499 90)
+			(at 144.78 67.3099 90)
 			(show_name no)
 			(do_not_autoplace no)
@@
 		)
 		(property "Footprint" ""
-			(at 127 120.65 0)
+			(at 148.59 67.31 0)
 			(hide yes)
 			(show_name no)
@@
 		)
 		(property "Datasheet" ""
-			(at 127 120.65 0)
+			(at 148.59 67.31 0)
 			(hide yes)
 			(show_name no)
@@
 		)
 		(property "Description" "Power symbol creates a global label with name \"+3V3\""
-			(at 127 120.65 0)
+			(at 148.59 67.31 0)
 			(hide yes)
 			(show_name no)
@@
 	(symbol
 		(lib_id "Connector_Generic:Conn_01x04")
-		(at 132.08 118.11 0)
+		(at 153.67 64.77 0)
 		(unit 1)
 		(body_style 1)
@@
 		(fields_autoplaced yes)
 		(property "Reference" "J1"
-			(at 134.62 118.1099 0)
+			(at 156.21 64.7699 0)
 			(show_name no)
 			(do_not_autoplace no)
@@
 		)
 		(property "Value" "Conn_01x04"
-			(at 134.62 120.6499 0)
+			(at 156.21 67.3099 0)
 			(show_name no)
 			(do_not_autoplace no)
@@
 		)
 		(property "Footprint" ""
-			(at 132.08 118.11 0)
+			(at 153.67 64.77 0)
 			(hide yes)
 			(show_name no)
@@
 		)
 		(property "Datasheet" ""
-			(at 132.08 118.11 0)
+			(at 153.67 64.77 0)
 			(hide yes)
 			(show_name no)
@@
 		)
 		(property "Description" "Generic connector, single row, 01x04, script generated (kicad-library-utils/schlib/autogen/connector/)"
-			(at 132.08 118.11 0)
+			(at 153.67 64.77 0)
 			(hide yes)
 			(show_name no)
@@
 	(symbol
 		(lib_id "power:GND")
-		(at 127 123.19 270)
+		(at 148.59 69.85 270)
 		(unit 1)
 		(body_style 1)
@@
 		(fields_autoplaced yes)
 		(property "Reference" "#PWR06"
-			(at 120.65 123.19 0)
+			(at 142.24 69.85 0)
 			(hide yes)
 			(show_name no)
@@
 		)
 		(property "Value" "GND"
-			(at 123.19 123.1899 90)
+			(at 144.78 69.8499 90)
 			(show_name no)
 			(do_not_autoplace no)
@@
 		)
 		(property "Footprint" ""
-			(at 127 123.19 0)
+			(at 148.59 69.85 0)
 			(hide yes)
 			(show_name no)
@@
 		)
 		(property "Datasheet" ""
-			(at 127 123.19 0)
+			(at 148.59 69.85 0)
 			(hide yes)
 			(show_name no)
@@
 		)
 		(property "Description" "Power symbol creates a global label with name \"GND\" , ground"
-			(at 127 123.19 0)
-			(hide yes)
-			(show_name no)
+			(at 148.59 69.85 0)
+			(hide yes)
+			(show_name no)

Commit message: Added io_connectors.kicad_sch and power_distribution.kicad_sch, and modified mcu_esp32.kicad_sch
Changed lines of the file:
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@@
 		)
 	)
-	(label "MISO"
+	(hierarchical_label "DSHOT_M1"
+		(shape input)
+		(at 127 77.47 0)
+		(effects
+			(font
+				(size 1.27 1.27)
+			)
+			(justify left)
+		)
+	)
+	(hierarchical_label "MOSI"
+		(shape input)
+		(at 127 100.33 0)
+		(effects
+			(font
+				(size 1.27 1.27)
+			)
+			(justify left)
+		)
+	)
+	(hierarchical_label "IMU_CS"
+		(shape input)
+		(at 127 72.39 0)
+		(effects
+			(font
+				(size 1.27 1.27)
+			)
+			(justify left)
+		)
+	)
+	(hierarchical_label "SPI_SCK"
+		(shape input)
+		(at 127 90.17 0)
+		(effects
+			(font
+				(size 1.27 1.27)
+			)
+			(justify left)
+		)
+	)
+	(hierarchical_label "DSHOT_M2"
+		(shape input)
+		(at 127 80.01 0)
+		(effects
+			(font
+				(size 1.27 1.27)
+			)
+			(justify left)
+		)
+	)
+	(hierarchical_label "DSHOT_M3"
+		(shape input)
+		(at 127 107.95 0)
+		(effects
+			(font
+				(size 1.27 1.27)
+			)
+			(justify left)
+		)
+	)
+	(hierarchical_label "DSHOT_M4"
+		(shape input)
+		(at 127 110.49 0)
+		(effects
+			(font
+				(size 1.27 1.27)
+			)
+			(justify left)
+		)
+	)
+	(hierarchical_label "MISO"
+		(shape input)
 		(at 127 92.71 0)
 		(effects
@@
 				(size 1.27 1.27)
 			)
-			(justify left bottom)
+			(justify left)
 		)
 	)
-	(label "DSHOT_M1"
-		(at 127 77.47 0)
-		(effects
-			(font
-				(size 1.27 1.27)
-			)
-			(justify left bottom)
-		)
-	)
-	(label "DSHOT_M2"
-		(at 127 80.01 0)
-		(effects
-			(font
-				(size 1.27 1.27)
-			)
-			(justify left bottom)
-		)
-	)
-	(label "SPI_SCK"
-		(at 127 90.17 0)
-		(effects
-			(font
-				(size 1.27 1.27)
-			)
-			(justify left bottom)
-		)
-	)
-	(label "IMU_CS"
-		(at 127 72.39 0)
-		(effects
-			(font
-				(size 1.27 1.27)
-			)
-			(justify left bottom)
-		)
-	)
-	(label "DSHOT_M3"
-		(at 127 107.95 0)
-		(effects
-			(font
-				(size 1.27 1.27)
-			)
-			(justify left bottom)
-		)
-	)
-	(label "MOSI"
-		(at 127 100.33 0)
-		(effects
-			(font
-				(size 1.27 1.27)
-			)
-			(justify left bottom)
-		)
-	)
-	(label "DSHOT_M4"
-		(at 127 110.49 0)
-		(effects
-			(font
-				(size 1.27 1.27)
-			)
-			(justify left bottom)
-		)
-	)
