File: electrical/kicad_project/io_connectors.kicad_sch (KiCad schematic)
At the start: 2 parts

Commit message: some changes
Changed lines of the file:
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@@
 	(wire
 		(pts
-			(xy 113.03 82.55) (xy 116.84 82.55)
+			(xy 111.76 82.55) (xy 116.84 82.55)
 		)
 		(stroke
@@
 	(symbol
 		(lib_id "power:PWR_FLAG")
-		(at 113.03 82.55 0)
+		(at 111.76 82.55 0)
 		(unit 1)
 		(body_style 1)
@@
 		(fields_autoplaced yes)
 		(property "Reference" "#FLG06"
-			(at 113.03 80.645 0)
+			(at 111.76 80.645 0)
 			(hide yes)
 			(show_name no)
@@
 		)
 		(property "Value" "+5V_DIRTY"
-			(at 113.03 77.47 0)
+			(at 111.76 77.47 0)
 			(show_name no)
 			(do_not_autoplace no)
@@
 		)
 		(property "Footprint" ""
-			(at 113.03 82.55 0)
+			(at 111.76 82.55 0)
 			(hide yes)
 			(show_name no)
@@
 		)
 		(property "Datasheet" ""
-			(at 113.03 82.55 0)
+			(at 111.76 82.55 0)
 			(hide yes)
 			(show_name no)
@@
 		)
 		(property "Description" "Special symbol for telling ERC where power comes from"
-			(at 113.03 82.55 0)
-			(hide yes)
-			(show_name no)
+			(at 111.76 82.55 0)
+			(hide yes)
+			(show_name no)
