File: electrical/kicad_project/sensors_imu.kicad_sch (KiCad schematic)
At the start: 4 parts, among them U1 BMI160

Commit message: some changes
Parts:
- added FB2: FerriteBead, symbol Device:FerriteBead
Connections:
- net +3V3: now also FB2.2; no longer C1.1, C2.2, R1.1, U1.5 (VDDIO), U1.8 (VDD)
- new net +3V3_IMU: C1.1, C2.2, FB2.1, R1.1, U1.5 (VDDIO), U1.8 (VDD)
Other:
- note added: "MECHANICAL: Soft-mount PCB with Silicone Grommets. Tune durometer to damp >100Hz motor noise without introducing low-frequency oscillation."
- note removed: "LAYOUT NOTE: Place 100nF caps < 2mm from VDD pins."
- moved on the sheet: R1

Commit message: new push
Parts:
- C1, C2: footprint (none) -> Capacitor_SMD:C_0402_1005Metric
- FB2: footprint (none) -> Inductor_SMD:L_0402_1005Metric
- R1: footprint (none) -> Resistor_SMD:R_0402_1005Metric
Changed lines of the file:
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@@
 			)
 		)
-		(property "Footprint" ""
+		(property "Footprint" "Capacitor_SMD:C_0402_1005Metric"
 			(at 125.73 63.5 0)
 			(hide yes)
@@
 			)
 		)
-		(property "Footprint" ""
+		(property "Footprint" "Resistor_SMD:R_0402_1005Metric"
 			(at 89.662 48.26 90)
 			(hide yes)
@@
 			)
 		)
-		(property "Footprint" ""
+		(property "Footprint" "Inductor_SMD:L_0402_1005Metric"
 			(at 79.502 34.29 90)
 			(hide yes)
@@
 			)
 		)
-		(property "Footprint" ""
+		(property "Footprint" "Capacitor_SMD:C_0402_1005Metric"
 			(at 121.92 71.12 0)
 			(hide yes)
