File: electrical/simulations/sim_pdn_ac/sim_pdn_ac.kicad_sch (KiCad schematic)
At the start: 0 parts

Commit message: PDN sim fixes and additions
Parts:
- added C1: 4.7uF, symbol Device:C
- added C2: 100nF, symbol Device:C
- added C3: 1uf, symbol Device:C
- added C4: 1uF, symbol Device:C
- added I1: 0.1, symbol Simulation_SPICE:IDC
- added L1: 0.5nH, symbol Device:L
- added L2: 0.3nH, symbol Device:L
- added L3: 0.4nH, symbol Device:L
- added L_TRACE1: 2nh, symbol Device:L
- added R1: 5m, symbol Device:R
- added R2: 20m, symbol Device:R
- added R3: 10m, symbol Device:R
- added R4: 0.22, symbol Device:R
- added V1: 3.3, symbol Simulation_SPICE:VDC
Connections:
- new net: L1.1, R1.2
- new net: C1.1, C3.1, C4.1, L_TRACE1.1, V1.1
- new net: C3.2, R3.1
- new net: L2.1, R2.2
- new net: C2.2, R2.1
- new net: C1.2, R1.1
- new net: C4.2, R4.1
- new net: L3.1, R3.2
- new net ESP32_VDD: C2.1, I1.1, L_TRACE1.2
- new net GND: I1.2, L1.2, L2.2, L3.2, R4.2, V1.2
